File: DingoPDM/BTS7008_2EPA.kicad_sch (KiCad schematic)
At the start: 13 parts, among them U9 BTS7008-2EPA

Commit message: Swapped to AMPSEAL 14 pins
Parts:
- renumbered C26 to C44, C27 to C45, C28 to C46, D12 to D36, R49 to R52, R50 to R53, R51 to R54, R52 to R55, R53 to R56, R54 to R57, R55 to R58, R56 to R59, U9 to U16
Changed lines of the file:
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@@
     (effects (font (size 1.27 1.27)) (justify right))
   )
-  (symbol (lib_id "Profet:BTS7008-2EPA") (at 118.11 85.09 0)
-    (in_bom yes) (on_board yes)
-    (property "Reference" "U9" (id 0) (at 128.27 80.8482 0))
+  (symbol (lib_id "Profet:BTS7008-2EPA") (at 118.11 85.09 0) (unit 1)
+    (in_bom yes) (on_board yes)
+    (property "Reference" "U16" (id 0) (at 128.27 80.8482 0))
     (property "Value" "BTS7008-2EPA" (id 1) (at 128.27 83.1596 0))
     (property "Footprint" "Profet:TDSO-14" (id 2) (at 118.11 85.09 0)
@@
     (pin "9")
   )
-  (symbol (lib_id "Device:R_Small_US") (at 92.71 92.71 270)
-    (in_bom yes) (on_board yes)
-    (property "Reference" "R49" (id 0) (at 92.71 87.503 90))
+  (symbol (lib_id "Device:R_Small_US") (at 92.71 92.71 270) (unit 1)
+    (in_bom yes) (on_board yes)
+    (property "Reference" "R52" (id 0) (at 92.71 87.503 90))
     (property "Value" "4.7K" (id 1) (at 92.71 89.8144 90))
     (property "Footprint" "Resistor_SMD:R_0805_2012Metric" (id 2) (at 92.71 92.71 0)
@@
     (pin "2")
   )
-  (symbol (lib_id "Device:R_Small_US") (at 92.71 95.25 270)
-    (in_bom yes) (on_board yes)
-    (property "Reference" "R50" (id 0) (at 92.71 100.33 90))
+  (symbol (lib_id "Device:R_Small_US") (at 92.71 95.25 270) (unit 1)
+    (in_bom yes) (on_board yes)
+    (property "Reference" "R53" (id 0) (at 92.71 100.33 90))
     (property "Value" "4.7K" (id 1) (at 92.71 97.79 90))
     (property "Footprint" "Resistor_SMD:R_0805_2012Metric" (id 2) (at 92.71 95.25 0)
@@
     (pin "2")
   )
-  (symbol (lib_id "Device:C_Small") (at 158.75 71.12 180)
-    (in_bom yes) (on_board yes)
-    (property "Reference" "C27" (id 0) (at 161.0868 69.9516 0)
+  (symbol (lib_id "Device:C_Small") (at 158.75 71.12 180) (unit 1)
+    (in_bom yes) (on_board yes)
+    (property "Reference" "C45" (id 0) (at 161.0868 69.9516 0)
       (effects (font (size 1.27 1.27)) (justify right))
     )
@@
     (pin "2")
   )
-  (symbol (lib_id "Device:C_Small") (at 146.05 71.12 180)
-    (in_bom yes) (on_board yes)
-    (property "Reference" "C26" (id 0) (at 148.3868 69.9516 0)
+  (symbol (lib_id "Device:C_Small") (at 146.05 71.12 180) (unit 1)
+    (in_bom yes) (on_board yes)
+    (property "Reference" "C44" (id 0) (at 148.3868 69.9516 0)
       (effects (font (size 1.27 1.27)) (justify right))
     )
@@
     (pin "2")
   )
-  (symbol (lib_id "Device:R_Small_US") (at 152.4 80.01 270)
-    (in_bom yes) (on_board yes)
-    (property "Reference" "R54" (id 0) (at 152.4 82.55 90))
+  (symbol (lib_id "Device:R_Small_US") (at 152.4 80.01 270) (unit 1)
+    (in_bom yes) (on_board yes)
+    (property "Reference" "R57" (id 0) (at 152.4 82.55 90))
     (property "Value" "47R 1/4W" (id 1) (at 152.4 85.09 90))
     (property "Footprint" "Resistor_SMD:R_1206_3216Metric" (id 2) (at 152.4 80.01 0)
@@
     (pin "2")
   )
-  (symbol (lib_id "power:GND") (at 158.75 80.01 0)
-    (in_bom yes) (on_board yes)
-    (property "Reference" "#PWR048" (id 0) (at 158.75 86.36 0)
+  (symbol (lib_id "power:GND") (at 158.75 80.01 0) (unit 1)
+    (in_bom yes) (on_board yes)
+    (property "Reference" "#PWR0140" (id 0) (at 158.75 86.36 0)
       (effects (font (size 1.27 1.27)) hide)
     )
@@
     (pin "1")
   )
-  (symbol (lib_id "Device:R_Small_US") (at 175.26 113.03 270)
-    (in_bom yes) (on_board yes)
-    (property "Reference" "R56" (id 0) (at 175.26 115.57 90))
+  (symbol (lib_id "Device:R_Small_US") (at 175.26 113.03 270) (unit 1)
+    (in_bom yes) (on_board yes)
+    (property "Reference" "R59" (id 0) (at 175.26 115.57 90))
     (property "Value" "4.7K" (id 1) (at 175.26 118.11 90))
     (property "Footprint" "Resistor_SMD:R_0805_2012Metric" (id 2) (at 175.26 113.03 0)
@@
     (pin "2")
   )
-  (symbol (lib_id "Device:C_Small") (at 181.61 115.57 180)
-    (in_bom yes) (on_board yes)
-    (property "Reference" "C28" (id 0) (at 184.15 115.57 0)
+  (symbol (lib_id "Device:C_Small") (at 181.61 115.57 180) (unit 1)
+    (in_bom yes) (on_board yes)
+    (property "Reference" "C46" (id 0) (at 184.15 115.57 0)
       (effects (font (size 1.27 1.27)) (justify right))
     )
@@
     (pin "2")
   )
-  (symbol (lib_id "Device:R_Small_US") (at 147.32 115.57 0)
-    (in_bom yes) (on_board yes)
-    (property "Reference" "R53" (id 0) (at 142.24 114.3 0)
+  (symbol (lib_id "Device:R_Small_US") (at 147.32 115.57 0) (unit 1)
+    (in_bom yes) (on_board yes)
+    (property "Reference" "R56" (id 0) (at 142.24 114.3 0)
       (effects (font (size 1.27 1.27)) (justify left))
     )
@@
     (pin "2")
   )
-  (symbol (lib_id "Device:R_Small_US") (at 154.94 113.03 270)
-    (in_bom yes) (on_board yes)
-    (property "Reference" "R55" (id 0) (at 154.94 115.57 90))
+  (symbol (lib_id "Device:R_Small_US") (at 154.94 113.03 270) (unit 1)
+    (in_bom yes) (on_board yes)
+    (property "Reference" "R58" (id 0) (at 154.94 115.57 90))
     (property "Value" "220K" (id 1) (at 154.94 118.11 90))
     (property "Footprint" "Resistor_SMD:R_0805_2012Metric" (id 2) (at 154.94 113.03 0)
@@
     (pin "2")
   )
-  (symbol (lib_id "Device:D_Zener_Small") (at 162.56 115.57 270)
-    (in_bom yes) (on_board yes)
-    (property "Reference" "D12" (id 0) (at 164.2872 114.4016 90)
+  (symbol (lib_id "Device:D_Zener_Small") (at 162.56 115.57 270) (unit 1)
+    (in_bom yes) (on_board yes)
+    (property "Reference" "D36" (id 0) (at 164.2872 114.4016 90)
       (effects (font (size 1.27 1.27)) (justify left))
     )
@@
     (pin "2")
   )
-  (symbol (lib_id "power:GND") (at 147.32 118.11 0)
-    (in_bom yes) (on_board yes)
-    (property "Reference" "#PWR047" (id 0) (at 147.32 124.46 0)
+  (symbol (lib_id "power:GND") (at 147.32 118.11 0) (unit 1)
+    (in_bom yes) (on_board yes)
+    (property "Reference" "#PWR0139" (id 0) (at 147.32 124.46 0)
       (effects (font (size 1.27 1.27)) hide)
     )
@@
     (pin "1")
   )
-  (symbol (lib_id "power:GND") (at 162.56 118.11 0)
-    (in_bom yes) (on_board yes)
-    (property "Reference" "#PWR049" (id 0) (at 162.56 124.46 0)
+  (symbol (lib_id "power:GND") (at 162.56 118.11 0) (unit 1)
+    (in_bom yes) (on_board yes)
+    (property "Reference" "#PWR0141" (id 0) (at 162.56 124.46 0)
       (effects (font (size 1.27 1.27)) hide)
     )
@@
     (pin "1")
   )
-  (symbol (lib_id "power:GND") (at 181.61 118.11 0)
-    (in_bom yes) (on_board yes)
-    (property "Reference" "#PWR050" (id 0) (at 181.61 124.46 0)
+  (symbol (lib_id "power:GND") (at 181.61 118.11 0) (unit 1)
+    (in_bom yes) (on_board yes)
+    (property "Reference" "#PWR0142" (id 0) (at 181.61 124.46 0)
       (effects (font (size 1.27 1.27)) hide)
     )
@@
     (pin "1")
   )
-  (symbol (lib_id "Device:R_Small_US") (at 102.87 100.33 90)
-    (in_bom yes) (on_board yes)
-    (property "Reference" "R51" (id 0) (at 102.87 95.25 90))
+  (symbol (lib_id "Device:R_Small_US") (at 102.87 100.33 90) (unit 1)
+    (in_bom yes) (on_board yes)
+    (property "Reference" "R54" (id 0) (at 102.87 95.25 90))
     (property "Value" "4.7K" (id 1) (at 102.87 97.79 90))
     (property "Footprint" "Resistor_SMD:R_0805_2012Metric" (id 2) (at 102.87 100.33 0)
@@
     (pin "2")
   )
-  (symbol (lib_id "Device:R_Small_US") (at 102.87 102.87 270)
-    (in_bom yes) (on_board yes)
-    (property "Reference" "R52" (id 0) (at 102.87 107.95 90))
+  (symbol (lib_id "Device:R_Small_US") (at 102.87 102.87 270) (unit 1)
+    (in_bom yes) (on_board yes)
+    (property "Reference" "R55" (id 0) (at 102.87 107.95 90))
     (property "Value" "4.7K" (id 1) (at 102.87 105.41 90))
     (property "Footprint" "Resistor_SMD:R_0805_2012Metric" (id 2) (at 102.87 102.87 0)

Commit message: Removed unused IRQs, added pd res on PF GPIO reset
Parts:
- renumbered C44 to C41, C45 to C42, C46 to C43
Changed lines of the file:
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@@
   (symbol (lib_id "Device:C_Small") (at 158.75 71.12 180) (unit 1)
     (in_bom yes) (on_board yes)
-    (property "Reference" "C45" (id 0) (at 161.0868 69.9516 0)
+    (property "Reference" "C42" (id 0) (at 161.0868 69.9516 0)
       (effects (font (size 1.27 1.27)) (justify right))
     )
@@
   (symbol (lib_id "Device:C_Small") (at 146.05 71.12 180) (unit 1)
     (in_bom yes) (on_board yes)
-    (property "Reference" "C44" (id 0) (at 148.3868 69.9516 0)
+    (property "Reference" "C41" (id 0) (at 148.3868 69.9516 0)
       (effects (font (size 1.27 1.27)) (justify right))
     )
@@
   (symbol (lib_id "power:GND") (at 158.75 80.01 0) (unit 1)
     (in_bom yes) (on_board yes)
-    (property "Reference" "#PWR0140" (id 0) (at 158.75 86.36 0)
+    (property "Reference" "#PWR0137" (id 0) (at 158.75 86.36 0)
       (effects (font (size 1.27 1.27)) hide)
     )
@@
   (symbol (lib_id "Device:C_Small") (at 181.61 115.57 180) (unit 1)
     (in_bom yes) (on_board yes)
-    (property "Reference" "C46" (id 0) (at 184.15 115.57 0)
+    (property "Reference" "C43" (id 0) (at 184.15 115.57 0)
       (effects (font (size 1.27 1.27)) (justify right))
     )
@@
   (symbol (lib_id "power:GND") (at 147.32 118.11 0) (unit 1)
     (in_bom yes) (on_board yes)
-    (property "Reference" "#PWR0139" (id 0) (at 147.32 124.46 0)
+    (property "Reference" "#PWR0136" (id 0) (at 147.32 124.46 0)
       (effects (font (size 1.27 1.27)) hide)
     )
@@
   (symbol (lib_id "power:GND") (at 162.56 118.11 0) (unit 1)
     (in_bom yes) (on_board yes)
-    (property "Reference" "#PWR0141" (id 0) (at 162.56 124.46 0)
+    (property "Reference" "#PWR0138" (id 0) (at 162.56 124.46 0)
       (effects (font (size 1.27 1.27)) hide)
     )
@@
   (symbol (lib_id "power:GND") (at 181.61 118.11 0) (unit 1)
     (in_bom yes) (on_board yes)
-    (property "Reference" "#PWR0142" (id 0) (at 181.61 124.46 0)
+    (property "Reference" "#PWR0139" (id 0) (at 181.61 124.46 0)
       (effects (font (size 1.27 1.27)) hide)
     )

Commit message: layout finished
Parts:
- renumbered C41 to C42, C42 to C43, C43 to C44, D36 to D35, R52 to R51, R53 to R52, R54 to R53, R55 to R54, R56 to R55, R57 to R56, R58 to R57, R59 to R58, U16 to U17
Changed lines of the file:
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@@
   (symbol (lib_id "Profet:BTS7008-2EPA") (at 118.11 85.09 0) (unit 1)
     (in_bom yes) (on_board yes)
-    (property "Reference" "U16" (id 0) (at 128.27 80.8482 0))
+    (property "Reference" "U17" (id 0) (at 128.27 80.8482 0))
     (property "Value" "BTS7008-2EPA" (id 1) (at 128.27 83.1596 0))
     (property "Footprint" "Profet:TDSO-14" (id 2) (at 118.11 85.09 0)
@@
   (symbol (lib_id "Device:R_Small_US") (at 92.71 92.71 270) (unit 1)
     (in_bom yes) (on_board yes)
-    (property "Reference" "R52" (id 0) (at 92.71 87.503 90))
+    (property "Reference" "R51" (id 0) (at 92.71 87.503 90))
     (property "Value" "4.7K" (id 1) (at 92.71 89.8144 90))
     (property "Footprint" "Resistor_SMD:R_0805_2012Metric" (id 2) (at 92.71 92.71 0)
@@
   (symbol (lib_id "Device:R_Small_US") (at 92.71 95.25 270) (unit 1)
     (in_bom yes) (on_board yes)
-    (property "Reference" "R53" (id 0) (at 92.71 100.33 90))
+    (property "Reference" "R52" (id 0) (at 92.71 100.33 90))
     (property "Value" "4.7K" (id 1) (at 92.71 97.79 90))
     (property "Footprint" "Resistor_SMD:R_0805_2012Metric" (id 2) (at 92.71 95.25 0)
@@
   (symbol (lib_id "Device:C_Small") (at 158.75 71.12 180) (unit 1)
     (in_bom yes) (on_board yes)
-    (property "Reference" "C42" (id 0) (at 161.0868 69.9516 0)
+    (property "Reference" "C43" (id 0) (at 161.0868 69.9516 0)
       (effects (font (size 1.27 1.27)) (justify right))
     )
@@
   (symbol (lib_id "Device:C_Small") (at 146.05 71.12 180) (unit 1)
     (in_bom yes) (on_board yes)
-    (property "Reference" "C41" (id 0) (at 148.3868 69.9516 0)
+    (property "Reference" "C42" (id 0) (at 148.3868 69.9516 0)
       (effects (font (size 1.27 1.27)) (justify right))
     )
@@
   (symbol (lib_id "Device:R_Small_US") (at 152.4 80.01 270) (unit 1)
     (in_bom yes) (on_board yes)
-    (property "Reference" "R57" (id 0) (at 152.4 82.55 90))
+    (property "Reference" "R56" (id 0) (at 152.4 82.55 90))
     (property "Value" "47R 1/4W" (id 1) (at 152.4 85.09 90))
     (property "Footprint" "Resistor_SMD:R_1206_3216Metric" (id 2) (at 152.4 80.01 0)
@@
   (symbol (lib_id "power:GND") (at 158.75 80.01 0) (unit 1)
     (in_bom yes) (on_board yes)
-    (property "Reference" "#PWR0137" (id 0) (at 158.75 86.36 0)
+    (property "Reference" "#PWR0138" (id 0) (at 158.75 86.36 0)
       (effects (font (size 1.27 1.27)) hide)
     )
@@
   (symbol (lib_id "Device:R_Small_US") (at 175.26 113.03 270) (unit 1)
     (in_bom yes) (on_board yes)
-    (property "Reference" "R59" (id 0) (at 175.26 115.57 90))
+    (property "Reference" "R58" (id 0) (at 175.26 115.57 90))
     (property "Value" "4.7K" (id 1) (at 175.26 118.11 90))
     (property "Footprint" "Resistor_SMD:R_0805_2012Metric" (id 2) (at 175.26 113.03 0)
@@
   (symbol (lib_id "Device:C_Small") (at 181.61 115.57 180) (unit 1)
     (in_bom yes) (on_board yes)
-    (property "Reference" "C43" (id 0) (at 184.15 115.57 0)
+    (property "Reference" "C44" (id 0) (at 184.15 115.57 0)
       (effects (font (size 1.27 1.27)) (justify right))
     )
@@
   (symbol (lib_id "Device:R_Small_US") (at 147.32 115.57 0) (unit 1)
     (in_bom yes) (on_board yes)
-    (property "Reference" "R56" (id 0) (at 142.24 114.3 0)
+    (property "Reference" "R55" (id 0) (at 142.24 114.3 0)
       (effects (font (size 1.27 1.27)) (justify left))
     )
@@
   (symbol (lib_id "Device:R_Small_US") (at 154.94 113.03 270) (unit 1)
     (in_bom yes) (on_board yes)
-    (property "Reference" "R58" (id 0) (at 154.94 115.57 90))
+    (property "Reference" "R57" (id 0) (at 154.94 115.57 90))
     (property "Value" "220K" (id 1) (at 154.94 118.11 90))
     (property "Footprint" "Resistor_SMD:R_0805_2012Metric" (id 2) (at 154.94 113.03 0)
@@
   (symbol (lib_id "Device:D_Zener_Small") (at 162.56 115.57 270) (unit 1)
     (in_bom yes) (on_board yes)
-    (property "Reference" "D36" (id 0) (at 164.2872 114.4016 90)
+    (property "Reference" "D35" (id 0) (at 164.2872 114.4016 90)
       (effects (font (size 1.27 1.27)) (justify left))
     )
@@
   (symbol (lib_id "power:GND") (at 147.32 118.11 0) (unit 1)
     (in_bom yes) (on_board yes)
-    (property "Reference" "#PWR0136" (id 0) (at 147.32 124.46 0)
+    (property "Reference" "#PWR0137" (id 0) (at 147.32 124.46 0)
       (effects (font (size 1.27 1.27)) hide)
     )
@@
   (symbol (lib_id "power:GND") (at 162.56 118.11 0) (unit 1)
     (in_bom yes) (on_board yes)
-    (property "Reference" "#PWR0138" (id 0) (at 162.56 124.46 0)
+    (property "Reference" "#PWR0139" (id 0) (at 162.56 124.46 0)
       (effects (font (size 1.27 1.27)) hide)
     )
@@
   (symbol (lib_id "power:GND") (at 181.61 118.11 0) (unit 1)
     (in_bom yes) (on_board yes)
-    (property "Reference" "#PWR0139" (id 0) (at 181.61 124.46 0)
+    (property "Reference" "#PWR0140" (id 0) (at 181.61 124.46 0)
       (effects (font (size 1.27 1.27)) hide)
     )
@@
   (symbol (lib_id "Device:R_Small_US") (at 102.87 100.33 90) (unit 1)
     (in_bom yes) (on_board yes)
-    (property "Reference" "R54" (id 0) (at 102.87 95.25 90))
+    (property "Reference" "R53" (id 0) (at 102.87 95.25 90))
     (property "Value" "4.7K" (id 1) (at 102.87 97.79 90))
     (property "Footprint" "Resistor_SMD:R_0805_2012Metric" (id 2) (at 102.87 100.33 0)
@@
   (symbol (lib_id "Device:R_Small_US") (at 102.87 102.87 270) (unit 1)
     (in_bom yes) (on_board yes)
-    (property "Reference" "R55" (id 0) (at 102.87 107.95 90))
+    (property "Reference" "R54" (id 0) (at 102.87 107.95 90))
     (property "Value" "4.7K" (id 1) (at 102.87 105.41 90))
     (property "Footprint" "Resistor_SMD:R_0805_2012Metric" (id 2) (at 102.87 102.87 0)

Commit message: Documentation cleanup
Parts:
- R51, R52, R53, R54, R58: value 4.7K -> 4.7k
- R55: value 1.2K -> 1.2k
- R57: value 220K -> 220k
Changed lines of the file:
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@@
       (effects (font (size 1.27 1.27)))
     )
-    (property "Value" "4.7K" (at 92.71 89.8144 90)
+    (property "Value" "4.7k" (at 92.71 89.8144 90)
       (effects (font (size 1.27 1.27)))
     )
@@
       (effects (font (size 1.27 1.27)) hide)
     )
-    (property "Datasheet" "~" (at 92.71 92.71 0)
+    (property "Datasheet" "" (at 92.71 92.71 0)
       (effects (font (size 1.27 1.27)) hide)
     )
@@
       (effects (font (size 1.27 1.27)))
     )
-    (property "Value" "4.7K" (at 92.71 97.79 90)
+    (property "Value" "4.7k" (at 92.71 97.79 90)
       (effects (font (size 1.27 1.27)))
     )
@@
       (effects (font (size 1.27 1.27)) hide)
     )
-    (property "Datasheet" "~" (at 92.71 95.25 0)
+    (property "Datasheet" "" (at 92.71 95.25 0)
       (effects (font (size 1.27 1.27)) hide)
     )
@@
       (effects (font (size 1.27 1.27)) hide)
     )
-    (property "Datasheet" "~" (at 158.75 71.12 0)
+    (property "Datasheet" "" (at 158.75 71.12 0)
       (effects (font (size 1.27 1.27)) hide)
     )
@@
       (effects (font (size 1.27 1.27)) hide)
     )
-    (property "Datasheet" "~" (at 146.05 71.12 0)
+    (property "Datasheet" "" (at 146.05 71.12 0)
       (effects (font (size 1.27 1.27)) hide)
     )
@@
       (effects (font (size 1.27 1.27)) hide)
     )
-    (property "Datasheet" "~" (at 152.4 80.01 0)
+    (property "Datasheet" "" (at 152.4 80.01 0)
       (effects (font (size 1.27 1.27)) hide)
     )
@@
       (effects (font (size 1.27 1.27)))
     )
-    (property "Value" "4.7K" (at 175.26 118.11 90)
+    (property "Value" "4.7k" (at 175.26 118.11 90)
       (effects (font (size 1.27 1.27)))
     )
@@
       (effects (font (size 1.27 1.27)) hide)
     )
-    (property "Datasheet" "~" (at 175.26 113.03 0)
+    (property "Datasheet" "" (at 175.26 113.03 0)
       (effects (font (size 1.27 1.27)) hide)
     )
@@
       (effects (font (size 1.27 1.27)) hide)
     )
-    (property "Datasheet" "~" (at 181.61 115.57 0)
+    (property "Datasheet" "" (at 181.61 115.57 0)
       (effects (font (size 1.27 1.27)) hide)
     )
@@
       (effects (font (size 1.27 1.27)) (justify left))
     )
-    (property "Value" "1.2K" (at 140.97 116.84 0)
+    (property "Value" "1.2k" (at 140.97 116.84 0)
       (effects (font (size 1.27 1.27)) (justify left))
     )
@@
       (effects (font (size 1.27 1.27)) hide)
     )
-    (property "Datasheet" "~" (at 147.32 115.57 0)
+    (property "Datasheet" "" (at 147.32 115.57 0)
       (effects (font (size 1.27 1.27)) hide)
     )
@@
       (effects (font (size 1.27 1.27)))
     )
-    (property "Value" "220K" (at 154.94 118.11 90)
+    (property "Value" "220k" (at 154.94 118.11 90)
       (effects (font (size 1.27 1.27)))
     )
@@
       (effects (font (size 1.27 1.27)) hide)
     )
-    (property "Datasheet" "~" (at 154.94 113.03 0)
+    (property "Datasheet" "" (at 154.94 113.03 0)
       (effects (font (size 1.27 1.27)) hide)
     )
@@
       (effects (font (size 1.27 1.27)) hide)
     )
-    (property "Datasheet" "~" (at 162.56 115.57 90)
+    (property "Datasheet" "" (at 162.56 115.57 90)
       (effects (font (size 1.27 1.27)) hide)
     )
@@
       (effects (font (size 1.27 1.27)))
     )
-    (property "Value" "4.7K" (at 102.87 97.79 90)
+    (property "Value" "4.7k" (at 102.87 97.79 90)
       (effects (font (size 1.27 1.27)))
     )
@@
       (effects (font (size 1.27 1.27)) hide)
     )
-    (property "Datasheet" "~" (at 102.87 100.33 0)
+    (property "Datasheet" "" (at 102.87 100.33 0)
       (effects (font (size 1.27 1.27)) hide)
     )
@@
       (effects (font (size 1.27 1.27)))
     )
-    (property "Value" "4.7K" (at 102.87 105.41 90)
+    (property "Value" "4.7k" (at 102.87 105.41 90)
       (effects (font (size 1.27 1.27)))
     )
@@
       (effects (font (size 1.27 1.27)) hide)
     )
-    (property "Datasheet" "~" (at 102.87 102.87 0)
-      (effects (font (size 1.27 1.27)) hide)
-    )
+    (property "Datasheet" "" (at 102.87 102.87 0)
+      (effects (font (size 1.27 1.27)) hide)
+    )

Commit message: V5 As Built
-Changed ADS1015 to MAX11613EUA+T due to supply issues
-Changed PCB to match JLCPCB 2oz rules
-Changed ON_SW input to 12V switched
-Switched to TagConnect TC2030
-Changed pin positions of GND, IN1, IN2
Other:
- title: (none) -> Dingo_PDM
Changed lines of the file:
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@@
 (kicad_sch (version 20230121) (generator eeschema)
   (paper "A4")
+  (title_block
+    (title "Dingo_PDM")
+    (date "2023-02-23")
+    (rev "v5")
+    (comment 3 "github.com/corygrant")
+    (comment 4 "Cory Grant")
+  )
   (junction (at 181.61 113.03) (diameter 0) (color 0 0 0 0)
   )

Commit message: Incorrect PN for some diodes and resistors
Parts:
- D35: Digi-Key_PN SZMMSZ4684T1GOSCT-ND -> 1727-5150-1-ND
Changed lines of the file:
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@@
       (effects (font (size 1.27 1.27)) hide)
     )
-    (property "Digi-Key_PN" "SZMMSZ4684T1GOSCT-ND" (at 162.56 115.57 0)
+    (property "Digi-Key_PN" "1727-5150-1-ND" (at 162.56 115.57 0)
       (effects (font (size 1.27 1.27)) hide)
     )
