File: DingoPDM/BTS700n_1EPP.kicad_sch (KiCad schematic)
At the start: 13 parts, among them U20 BTS700n-1EPP

Commit message: Documentation cleanup
Parts:
- D40: Status Active -> (none)
- R71, R72, R76: value 4.7K -> 4.7k
- R73: value 1.2K -> 1.2k
- R75: value 220K -> 220k
Changed lines of the file:
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@@
       (effects (font (size 1.27 1.27)))
     )
-    (property "Value" "4.7K" (at 96.52 87.2744 90)
+    (property "Value" "4.7k" (at 96.52 87.2744 90)
       (effects (font (size 1.27 1.27)))
     )
@@
       (effects (font (size 1.27 1.27)) hide)
     )
-    (property "Datasheet" "~" (at 96.52 90.17 0)
+    (property "Datasheet" "" (at 96.52 90.17 0)
       (effects (font (size 1.27 1.27)) hide)
     )
@@
       (effects (font (size 1.27 1.27)))
     )
-    (property "Value" "4.7K" (at 96.52 95.25 90)
+    (property "Value" "4.7k" (at 96.52 95.25 90)
       (effects (font (size 1.27 1.27)))
     )
@@
       (effects (font (size 1.27 1.27)) hide)
     )
-    (property "Datasheet" "~" (at 96.52 92.71 0)
+    (property "Datasheet" "" (at 96.52 92.71 0)
       (effects (font (size 1.27 1.27)) hide)
     )
@@
       (effects (font (size 1.27 1.27)) hide)
     )
-    (property "Datasheet" "~" (at 162.56 68.58 0)
+    (property "Datasheet" "" (at 162.56 68.58 0)
       (effects (font (size 1.27 1.27)) hide)
     )
@@
       (effects (font (size 1.27 1.27)) hide)
     )
-    (property "Datasheet" "~" (at 149.86 68.58 0)
+    (property "Datasheet" "" (at 149.86 68.58 0)
       (effects (font (size 1.27 1.27)) hide)
     )
@@
       (effects (font (size 1.27 1.27)) hide)
     )
-    (property "Datasheet" "~" (at 156.21 77.47 0)
+    (property "Datasheet" "" (at 156.21 77.47 0)
       (effects (font (size 1.27 1.27)) hide)
     )
@@
       (effects (font (size 1.27 1.27)) hide)
     )
-    (property "Datasheet" "~" (at 185.42 99.06 0)
+    (property "Datasheet" "" (at 185.42 99.06 0)
       (effects (font (size 1.27 1.27)) hide)
     )
@@
       (effects (font (size 1.27 1.27)))
     )
-    (property "Value" "4.7K" (at 179.07 115.57 90)
+    (property "Value" "4.7k" (at 179.07 115.57 90)
       (effects (font (size 1.27 1.27)))
     )
@@
       (effects (font (size 1.27 1.27)) hide)
     )
-    (property "Datasheet" "~" (at 179.07 110.49 0)
+    (property "Datasheet" "" (at 179.07 110.49 0)
       (effects (font (size 1.27 1.27)) hide)
     )
@@
       (effects (font (size 1.27 1.27)) hide)
     )
-    (property "Datasheet" "~" (at 185.42 113.03 0)
+    (property "Datasheet" "" (at 185.42 113.03 0)
       (effects (font (size 1.27 1.27)) hide)
     )
@@
       (effects (font (size 1.27 1.27)) (justify left))
     )
-    (property "Value" "1.2K" (at 144.78 114.3 0)
+    (property "Value" "1.2k" (at 144.78 114.3 0)
       (effects (font (size 1.27 1.27)) (justify left))
     )
@@
       (effects (font (size 1.27 1.27)) hide)
     )
-    (property "Datasheet" "~" (at 151.13 113.03 0)
+    (property "Datasheet" "" (at 151.13 113.03 0)
       (effects (font (size 1.27 1.27)) hide)
     )
@@
       (effects (font (size 1.27 1.27)))
     )
-    (property "Value" "220K" (at 158.75 115.57 90)
+    (property "Value" "220k" (at 158.75 115.57 90)
       (effects (font (size 1.27 1.27)))
     )
@@
       (effects (font (size 1.27 1.27)) hide)
     )
-    (property "Datasheet" "~" (at 158.75 110.49 0)
+    (property "Datasheet" "" (at 158.75 110.49 0)
       (effects (font (size 1.27 1.27)) hide)
     )
@@
       (effects (font (size 1.27 1.27)) hide)
     )
-    (property "Datasheet" "~" (at 166.37 113.03 90)
+    (property "Datasheet" "" (at 166.37 113.03 90)
       (effects (font (size 1.27 1.27)) hide)
     )
@@
       (effects (font (size 1.524 1.524)) (justify left) hide)
     )
-    (property "MPN" "" (at 177.8 104.14 0)
-      (effects (font (size 1.524 1.524)) (justify left) hide)
-    )
-    (property "Category" "" (at 180.34 104.14 0)
-      (effects (font (size 1.524 1.524)) (justify left) hide)
-    )
-    (property "Family" "" (at 182.88 104.14 0)
-      (effects (font (size 1.524 1.524)) (justify left) hide)
-    )
-    (property "DK_Datasheet_Link" "" (at 185.42 104.14 0)
-      (effects (font (size 1.524 1.524)) (justify left) hide)
-    )
-    (property "DK_Detail_Page" "" (at 187.96 104.14 0)
-      (effects (font (size 1.524 1.524)) (justify left) hide)
-    )
-    (property "Description" "" (at 190.5 104.14 0)
-      (effects (font (size 1.524 1.524)) (justify left) hide)
-    )
-    (property "Manufacturer" "" (at 193.04 104.14 0)
-      (effects (font (size 1.524 1.524)) (justify left) hide)
-    )
-    (property "Status" "Active" (at 195.58 104.14 0)
-      (effects (font (size 1.524 1.524)) (justify left) hide)
-    )

Commit message: V5 As Built
-Changed ADS1015 to MAX11613EUA+T due to supply issues
-Changed PCB to match JLCPCB 2oz rules
-Changed ON_SW input to 12V switched
-Switched to TagConnect TC2030
-Changed pin positions of GND, IN1, IN2
Other:
- title: (none) -> Dingo_PDM
Changed lines of the file:
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@@
 (kicad_sch (version 20230121) (generator eeschema)
   (paper "A4")
+  (title_block
+    (title "Dingo_PDM")
+    (date "2023-02-23")
+    (rev "v5")
+    (comment 3 "github.com/corygrant")
+    (comment 4 "Cory Grant")
+  )
   (junction (at 185.42 96.52) (diameter 0) (color 0 0 0 0)
   )

Commit message: Incorrect PN for some diodes and resistors
Parts:
- D41: Digi-Key_PN SZMMSZ4684T1GOSCT-ND -> 1727-5150-1-ND
Changed lines of the file:
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@@
       (effects (font (size 1.27 1.27)) hide)
     )
-    (property "Digi-Key_PN" "SZMMSZ4684T1GOSCT-ND" (at 166.37 113.03 0)
+    (property "Digi-Key_PN" "1727-5150-1-ND" (at 166.37 113.03 0)
       (effects (font (size 1.27 1.27)) hide)
     )
