File: DingoPDM/DigIn.kicad_sch (KiCad schematic)
At the start: 6 parts

Commit message: Small edits
Parts:
- R10, R9: value 4.7k -> 4.7K
Changed lines of the file:
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@@
       (effects (font (size 1.27 1.27)))
     )
-    (property "Value" "4.7k" (at 34.29 29.4894 90)
+    (property "Value" "4.7K" (at 34.29 29.4894 90)
       (effects (font (size 1.27 1.27)))
     )
@@
       (effects (font (size 1.27 1.27)))
     )
-    (property "Value" "4.7k" (at 34.29 58.0644 90)
+    (property "Value" "4.7K" (at 34.29 58.0644 90)
       (effects (font (size 1.27 1.27)))
     )
