File: DingoPDM/HighCurrentDrivers.kicad_sch (KiCad schematic)
At the start: 4 parts, among them U7 LM324

Commit message: Update JLC part numbers for in stock ones
Parts:
- U7: LCSC C7944 -> C7942
Changed lines of the file:
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@@
       (effects (font (size 1.27 1.27)) hide)
     )
-    (property "LCSC" "C7944" (at 139.065 58.42 0)
+    (property "LCSC" "C7942" (at 139.065 58.42 0)
       (effects (font (size 1.27 1.27)) hide)
     )
@@
       (effects (font (size 1.27 1.27)) hide)
     )
-    (property "LCSC" "C7944" (at 139.7 82.55 0)
+    (property "LCSC" "C7942" (at 139.7 82.55 0)
       (effects (font (size 1.27 1.27)) hide)
     )
@@
       (effects (font (size 1.27 1.27)) hide)
     )
-    (property "LCSC" "C7944" (at 234.95 40.005 0)
+    (property "LCSC" "C7942" (at 234.95 40.005 0)
       (effects (font (size 1.27 1.27)) hide)
     )

Commit message: Updated to Kicad 8
Parts:
- renumbered C41 to C21, R8 to R11, R8 to R12
