File: DingoPDM/Connectors.kicad_sch (KiCad schematic)
At the start: 13 parts, among them J1 RedCubeTerminal, J2 RedCubeTerminal, J3 Conn_01x12, J5 USB_C_Receptacle_USB2.0

Commit message: move footprints to project library
Parts:
- J1, J2: footprint RedCube:M6_Hole_8Pin_7461084 -> dingoPDM:M6_Hole_8Pin_7461084
- J3: footprint Deutsch_DT:DT15-12PA -> dingoPDM:DT15-12PA
Changed lines of the file:
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@@
 			)
 		)
-		(property "Footprint" "RedCube:M6_Hole_8Pin_7461084"
+		(property "Footprint" "dingoPDM:M6_Hole_8Pin_7461084"
 			(at 22.86 31.75 0)
 			(effects
@@
 			)
 		)
-		(property "Footprint" "Deutsch_DT:DT15-12PA"
+		(property "Footprint" "dingoPDM:DT15-12PA"
 			(at 106.68 56.515 0)
 			(effects
@@
 			)
 		)
-		(property "Footprint" "RedCube:M6_Hole_8Pin_7461084"
+		(property "Footprint" "dingoPDM:M6_Hole_8Pin_7461084"
 			(at 31.75 34.29 0)
 			(effects

Commit message: docs - add iboms
Parts:
- J1, J2: LCSC (none) -> C6828431
- J3: LCSC (none) -> C5341788
- J5: LCSC (none) -> C7095263
Changed lines of the file:
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@@
 			)
 		)
-		(property "LCSC" ""
+		(property "LCSC" "C6828431"
 			(at 22.86 31.75 0)
 			(effects
@@
 			)
 		)
-		(property "LCSC" ""
+		(property "LCSC" "C5341788"
 			(at 106.68 56.515 0)
 			(effects
@@
 			)
 		)
-		(property "LCSC" ""
+		(property "LCSC" "C6828431"
 			(at 31.75 34.29 0)
 			(effects
@@
 			(at 31.115 153.67 0)
 			(effects
+				(font
+					(size 1.27 1.27)
+				)
+				(hide yes)
+			)
+		)
+		(property "LCSC" "C7095263"
+			(at 31.115 153.67 0)
+			(effects
